File: hardware/kicad/xiamocon.kicad_pcb (KiCad board)
At the start: 2 copper layers, 100 x 50 mm, 75 parts, among them J1 JST S2B-PH-SM4-TB, J2 Conn_01x02, J3 Micro_SD_Card_Det_Hirose_DM3AT, J4 Hong Cheng HC-PM254-5.0H-2x10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, Q1 IRLML6344TRPBF, Q2 IRLML6344TRPBF, Q3 IRLML2246TRPBF, Q4 IRLML2246TRPBF, Q5 IRLML2246TRPBF, SW1 GT-TC018A-H0375-L1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

Commit message: PCB fixed
Parts:
- removed R10: 100k, Resistor_SMD:R_0402_1005Metric
- added C12: 1u, Capacitor_SMD:C_0603_1608Metric, F.Cu at (59.2, 69.2)
- added C13: 100n, Capacitor_SMD:C_0402_1005Metric, F.Cu at (123.8, 92.1)
- added C14: 100n, Capacitor_SMD:C_0402_1005Metric, F.Cu at (122.3, 95.0)
- added C15: 100n, Capacitor_SMD:C_0402_1005Metric, F.Cu at (53.7, 72.5)
- added C16: 1nF, Capacitor_SMD:C_0402_1005Metric, F.Cu at (59.5, 72.5)
- added G***: LOGO, LOGO, B.Cu at (147.6, 64.9)
- added Q6: BSS138W, Package_TO_SOT_SMD:SOT-323_SC-70, F.Cu at (98.8, 70.6)
- added Q7: BSS138W, Package_TO_SOT_SMD:SOT-323_SC-70, F.Cu at (103.8, 70.6)
- added Q8: BSS84W, Package_TO_SOT_SMD:SOT-323_SC-70, F.Cu at (119.9, 97.0)
- added Q9: BSS138W, Package_TO_SOT_SMD:SOT-323_SC-70, F.Cu at (124.7, 97.5)
- added R11: 100k, Resistor_SMD:R_0402_1005Metric, F.Cu at (75.4, 76.1)
- added R31: 100k, Resistor_SMD:R_0402_1005Metric, F.Cu at (100.7, 70.7)
- added R32: 100k, Resistor_SMD:R_0402_1005Metric, F.Cu at (105.7, 70.7)
- added R33: 0, Resistor_SMD:R_0402_1005Metric, F.Cu at (96.9, 70.7)
- added R34: 0, Resistor_SMD:R_0402_1005Metric, F.Cu at (101.9, 70.7)
- added R35: 0, Resistor_SMD:R_0402_1005Metric, F.Cu at (122.0, 89.1)
- added R36: 0, Resistor_SMD:R_0402_1005Metric, F.Cu at (120.0, 89.1)
- added R37: 10k, Resistor_SMD:R_0402_1005Metric, F.Cu at (121.8, 97.8)
- added R38: 10k, Resistor_SMD:R_0402_1005Metric, F.Cu at (122.3, 96.2)
- added R39: 100k, Resistor_SMD:R_0402_1005Metric, F.Cu at (124.5, 95.0)
- added R40: 100k, Resistor_SMD:R_0402_1005Metric, F.Cu at (119.9, 94.5)
- added R43: 22k, Resistor_SMD:R_0402_1005Metric, F.Cu at (60.6, 69.7)
- added R44: 22k, Resistor_SMD:R_0402_1005Metric, F.Cu at (59.4, 71.4)
- added TP1: PWAMP_CE, TestPoint:TestPoint_Pad_D1.5mm, F.Cu at (55.2, 78.0)
- added TP2: PWAMP_CE, TestPoint:TestPoint_Pad_D1.5mm, F.Cu at (128.5, 72.9)
- added TP3: PWAMP_CE, TestPoint:TestPoint_Pad_D1.5mm, F.Cu at (79.1, 57.8)
- added TP5: PWAMP_CE, TestPoint:TestPoint_Pad_D1.5mm, F.Cu at (59.6, 74.8)
- added TP6: PWAMP_CE, TestPoint:TestPoint_Pad_D1.5mm, F.Cu at (79.9, 86.0)
- added U7: ADC101C027CIMK, Package_TO_SOT_SMD:SOT-23-6, F.Cu at (121.2, 91.7)
- C8: value 47u -> 10u
- C9: value 10u -> 1u
- D5, D9: footprint LED_SMD:LED_0402_1005Metric -> LED_SMD:LED_0402_1005Metric_Pad0.77x0.64mm_HandSolder
- Q1, Q2: value IRLML6344TRPBF -> BSS138W; footprint Package_TO_SOT_SMD:SOT-23 -> Package_TO_SOT_SMD:SOT-323_SC-70
- Q5: value IRLML2246TRPBF -> BSS138W; footprint Package_TO_SOT_SMD:SOT-23 -> Package_TO_SOT_SMD:SOT-323_SC-70
- R20: value 22k -> 0
- R21, R8: footprint Resistor_SMD:R_0402_1005Metric -> Resistor_SMD:R_0402_1005Metric_Pad0.72x0.64mm_HandSolder
- R29, R30: value 10k -> 4.7k
- U4: value HT82V73A -> LM4890; footprint shpc_ic:SOIC-8_with_Thermal_Hole -> Package_SO:MSOP-8_3x3mm_P0.65mm
- moved C9 9.61 mm to (57.5, 76.3), turned to 90 degrees
- moved C8 7.04 mm to (53.2, 73.9)
- moved D4 2.12 mm to (73.1, 81.4), turned to 180 degrees
- moved R22 1.59 mm to (55.0, 75.3)
- moved R7 1.09 mm to (135.9, 72.1)
- moved Q1 1.00 mm to (81.9, 57.6), turned to -90 degrees
- moved Q5 0.89 mm to (68.7, 81.8)
- moved R5 0.89 mm to (136.4, 73.8)
- moved U4 0.83 mm to (56.6, 71.4), turned to 90 degrees
- moved J2 0.76 mm to (55.4, 63.0), turned to 0 degrees
- moved C4 0.57 mm to (120.7, 83.9)
- moved Q4 0.46 mm to (123.4, 85.0), turned to -90 degrees
- moved Q2 0.18 mm to (132.9, 72.9), turned to 180 degrees
- moved Q3 0.08 mm to (125.2, 74.2), turned to -90 degrees
Connections:
- C8 pad 1: GND -> VANL
- C8 pad 2: VANL -> GND
- C9 pad 2: Net-(U4-VREF) -> Net-(U4-+IN)
- D4 pad 1: /IOEX_MUTE -> /SPK_MUTE_N
- J4 pad 12: /I2C_SDA -> Net-(J4-Pin_12)
- J4 pad 13: /I2C_SCL -> Net-(J4-Pin_13)
- J4 pad 19: /SPK_MUTE -> /SPK_MUTE_N
- Q1 pad 1: Net-(Q1-D) -> Net-(D1-A)
- Q1 pad 2: Net-(D1-A) -> GND
- Q1 pad 3: GND -> Net-(Q1-D)
- Q2 pad 1: Net-(Q2-D) -> Net-(Q2-G)
- Q2 pad 2: Net-(Q2-G) -> /PERI_EN_N
- Q2 pad 3: /PERI_EN_N -> Net-(Q2-D)
- Q3 pad 1: VPERI -> Net-(Q2-D)
- Q3 pad 2: Net-(Q2-D) -> +3V3
- Q3 pad 3: +3V3 -> VPERI
- Q4 pad 1: /+BAT -> Net-(Q4-D)
- Q4 pad 2: Net-(Q4-G) -> VCOM
- Q4 pad 3: VCOM -> /+BAT
- Q5 pad 1: Net-(D4-A) -> /IOEX_MUTE_N
- Q5 pad 2: /SPK_MUTE -> GND
- Q5 pad 3: Net-(Q5-S) -> Net-(D4-A)
- R22 pad 1: Net-(Q5-S) -> VANL
- R22 pad 2: VANL -> Net-(D4-A)
- R9 pad 2: Net-(Q4-G) -> Net-(Q4-D)
- RV1 pad 2A: Net-(U4-IN) -> Net-(C12-Pad1)
- U4 pad 1: Net-(J2-Pin_2) -> Net-(D4-A)
- U4 pad 2: Net-(U4-IN) -> Net-(U4-+IN)
- U4 pad 3: Net-(U4-VREF) -> Net-(U4-+IN)
- U4 pad 4: GND -> Net-(U4--IN)
- U4 pad 5: Net-(Q5-S) -> Net-(J2-Pin_2)
- U4 pad 6: unconnected-(U4-NC-Pad6) -> VANL
- U4 pad 7: Net-(J2-Pin_1) -> GND
- U4 pad 8: VANL -> Net-(J2-Pin_1)
- U5 pad 10: /IOEX_MUTE -> /IOEX_MUTE_N
Routing:
- net VPERI: track 154.4 -> 185.1 mm, vias 4 -> 8
- net /SPK_MUTE: track 26.2 -> 0.00 mm
- net Net-(D4-A): track 2.29 -> 24.8 mm, vias 0 -> 2
- net /SPK_MUTE_N: track 0.00 -> 22.3 mm
- net Net-(U4-IN): track 21.0 -> 0.00 mm, vias 1 -> 0
- net Net-(C12-Pad1): track 0.00 -> 20.0 mm, vias 0 -> 1
- net Net-(Q5-S): track 18.3 -> 0.00 mm, vias 2 -> 0
- net Net-(J4-Pin_12): track 0.00 -> 17.8 mm
- net /+BAT: track 45.7 -> 61.0 mm, vias 0 -> 2
- net Net-(Q8-G): track 0.00 -> 11.0 mm
- net /I2C_SCL: track 117.2 -> 127.6 mm, vias 4 -> 5
- net VANL: track 32.1 -> 41.1 mm
- net Net-(J4-Pin_13): track 0.00 -> 8.96 mm
- net Net-(U7-V_{IN}): track 0.00 -> 7.82 mm
- net Net-(U4--IN): track 0.00 -> 7.02 mm
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Other:
- board text added: "3V3"
- board text added: "AUD"
- board text added: "EX0"
- board text added: "EX1"
- board text added: "EX2"
- board text added: "EX3"
- board text added: "GP0"
- board text added: "MIS"
- board text added: "MOS"
- board text added: "MUT"
- board text added: "SCL"
- board text added: "SDA"
- board text added: "VBU"
- board text added: "VCO"
- board text added: "VPE"
- board text removed: "Xiaonsole"
