File: hardware/kicad/xiamocon.kicad_sch (KiCad schematic)
At the start: 105 parts, among them J1 JST S2B-PH-SM4-TB, J2 Conn_01x02, J3 Micro_SD_Card_Det_Hirose_DM3AT, J4 Hong Cheng HC-PM254-5.0H-2x10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, Q1 BSS138W, Q2 BSS138W, Q3 IRLML2246TRPBF, Q4 IRLML2246TRPBF, Q5 BSS138W, Q6 BSS138W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

Commit message: PCB fixed
Parts:
- removed R41, R42: 0, Resistor_SMD:R_0402_1005Metric, symbol Device:R_Small
- removed TP4: PWAMP_CE, TestPoint:TestPoint_Pad_D1.5mm, symbol Connector:TestPoint_Small
- C16: footprint Capacitor_SMD:C_0603_1608Metric -> Capacitor_SMD:C_0402_1005Metric
Connections:
- net +3V3: no longer R35.1
- net VPERI: now also C13.2, R35.1, U7.1 (V_{A})
- net IOEX_MUTE renamed IOEX_MUTE_N
- net IOEX_MUTE_N: now also Q5.1 (G); no longer D4.1 (K)
- net SPK_MUTE renamed SPK_MUTE_N
- net SPK_MUTE_N: now also D4.1 (K); no longer Q5.1 (G)
Other:
- moved on the sheet: C13, C14, C5, Q8, Q9, R35, R36, R37, R38, R39, R40, U2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
