File: hardware/kicad/xiamocon.kicad_sch (KiCad schematic)
At the start: 109 parts, among them J1 FG PH-2AWT, J2 Conn_01x02, J3 Micro_SD_Card_Det_Hirose_DM3AT, J4 HC-PM254-5.0H-2x10PS, Q1 BSS138W, Q2 BSS138W, Q3 IRLML2246TRPBF, Q4 IRLML2246TRPBF, Q5 BSS138W, Q6 BSS138W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

Commit message: pcb rev.2 part changed
Parts:
- Q8: LCSC C42456334 -> C919394; URL https://www.lcsc.com/product-detail/C42456334.html -> https://www.lcsc.com/product-detail/C919394.html
Changed lines of the file:
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@@
 			)
 		)
-		(property "LCSC" "C42456334"
+		(property "LCSC" "C919394"
 			(at 276.86 49.53 90)
 			(effects
@@
 			)
 		)
-		(property "URL" "https://www.lcsc.com/product-detail/C42456334.html"
+		(property "URL" "https://www.lcsc.com/product-detail/C919394.html"
 			(at 276.86 49.53 90)
 			(effects
