File: hardware/kicad/xiamocon.kicad_sch (KiCad schematic)
At the start: 109 parts, among them J1 FG PH-2AWT, J2 Conn_01x02, J3 Micro_SD_Card_Det_Hirose_DM3AT, J4 HC-PM254-5.0H-2x10PS, Q1 BSS138W, Q2 BSS138W, Q3 IRLML2246TRPBF, Q4 IRLML2246TRPBF, Q5 BSS138W, Q6 BSS138W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

Commit message: fix: schematic
Parts:
- R12: now not fitted
- R29, R30: value 4.7k -> 2.2k; LCSC C25900 -> C25879; URL https://www.lcsc.com/product-detail/C25900.html -> https://www.lcsc.com/product-detail/C25879.html
Changed lines of the file:
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@@
 		(in_bom yes)
 		(on_board yes)
-		(dnp no)
+		(dnp yes)
 		(property "Reference" "R12"
 			(at 310.388 121.158 0)
@@
 			)
 		)
-		(property "Value" "4.7k"
+		(property "Value" "2.2k"
 			(at 74.93 31.75 0)
 			(effects
@@
 			)
 		)
-		(property "LCSC" "C25900"
+		(property "LCSC" "C25879"
 			(at 74.93 29.21 0)
 			(effects
@@
 			)
 		)
-		(property "URL" "https://www.lcsc.com/product-detail/C25900.html"
+		(property "URL" "https://www.lcsc.com/product-detail/C25879.html"
 			(at 74.93 29.21 0)
 			(effects
@@
 			)
 		)
-		(property "Value" "4.7k"
+		(property "Value" "2.2k"
 			(at 82.55 31.75 0)
 			(effects
@@
 			)
 		)
-		(property "LCSC" "C25900"
+		(property "LCSC" "C25879"
 			(at 82.55 29.21 0)
 			(effects
@@
 			)
 		)
-		(property "URL" "https://www.lcsc.com/product-detail/C25900.html"
+		(property "URL" "https://www.lcsc.com/product-detail/C25879.html"
 			(at 82.55 29.21 0)
 			(effects
